Commit message: Upated URDF files to rotate to vertical and move up 1 metre from ground plane

File: braccio_description/urdf/braccio_planning_model.urdf (robot description, URDF)
Before this commit: robot kr5, 9 links, 8 joints
Links:
- link link_2: geometry collision mesh filename=package://braccio_description/stl/braccio_shoulder.stl scale=0.001 0.001 0.00124; visual mesh filename=package://braccio_description/stl/braccio_shoulder.stl scale=0.001 0.001 0.00124
- link link_3: geometry collision mesh filename=package://braccio_description/stl/braccio_elbow.stl scale=0.001 0.001 0.00124; visual mesh filename=package://braccio_description/stl/braccio_elbow.stl scale=0.001 0.001 0.00124
Joints:
- joint elbow_joint: origin xyz=0 0 0.125 rpy=-1.5708 0 0 -> xyz=0 0 0.155 rpy=-1.5708 0 0
- joint world_joint: origin xyz=0.0 0.0 0.0 rpy=0.0 0.0 0.0 -> xyz=0.0 0.0 1.0 rpy=1.58 0.0 3.14
- joint wrist_pitch_joint: origin xyz=0 0 0.125 rpy=-1.5708 0 0 -> xyz=0 0 0.155 rpy=-1.5708 0 0
